File: PCB_Sensor_Stick/SensorStick.sch (EAGLE design)
At the start: 16 parts, among them IC1 SAM-M8Q-0-10, IC2 STM32L412RBT6P, IC3 DPS310XTSA1, IC4 SX1276IMLTRT, IC5 BMI085, J1 USB4160-03-0170-C, U1 4525DO-DS5AI001DP

Commit message: updated sch
Parts:
- added C10, C11, C6, C8: 0.1uF, SparkFun-Capacitors:0.1UF-0402-6.3V-10%-X7R
- added C12: 10uF, SparkFun-Capacitors:10UF-0603-6.3V-20%
- added C13: 0.22uF, SparkFun-Capacitors:0.22UF-0603-25V-10%
- added C7, C9: 1.0uF, SparkFun-Capacitors:1.0UF-0402-16V-10%
- added D1: SML-P12VTT86, ce-capstone:SML-P12VTT86
- added IC6: IIS2MDCTR, IIS2MDCTR:IIS2MDCTR
- added R3: 1KOHM-0402-1/16W-1%, SparkFun-Resistors:1KOHM-0402-1/16W-1%
- added U$1: STPS1L30A, ce-capstone:STPS1L30A
- added U2: LD39050PU33R, ce-capstone:LD39050PU33R
Connections:
- new net 5V: C6.1, C7.1, U$1.C, U2.EN, U2.VIN
- new net 5V_IN: U$1.A
- new net GPIO_EXTI4: IC2.PA4, IC6.INT/DRDY
- new net N$5: D1.A, R3.1
- new net N$6: C10.1, IC6.VDD_IO
- new net N$7: C13.1, IC6.C1
- net 3V3: now also C11.1, C12.1, C8.1, C9.1, IC6.VDD, R3.2, U2.VOUT
- net GND: now also C10.2, C11.2, C12.2, C13.2, C6.2, C7.2, C8.2, C9.2, D1.C, IC6.CS, IC6.GND_1, IC6.GND_2, U2.GND
- net I2C1_SCL: now also IC6.SCL/SPC
- net I2C1_SDA: now also IC6.SDA/SDI/SDO
