File: PCB_Sensor_Stick/SensorStick.sch (EAGLE design)
At the start: 31 parts, among them IC1 SAM-M8Q-0-10, IC2 STM32L412RBT6P, IC3 DPS310XTSA1, IC4 SX1276IMLTRT, IC5 BMI085, IC6 IIS2MDCTR, J1 USB4160-03-0230-C, U1 4525DO-DS5AI001DP, U2 LD39050PU33R

Commit message: Jesus- Up to date PCB sch/layout
Parts:
- removed FB1, FB2: BLM15HD102SN1, BLM15HD102SN1:BLM15HD102SN1
- removed IC1: SAM-M8Q-0-10, SAM-M8Q-0-10:SAM-M8Q-0-10
- removed IC3: DPS310XTSA1, DPS310XTSA1:DPS310XTSA1
- removed IC4: SX1276IMLTRT, SX1276IMLTRT:SX1276IMLTRT
- removed IC5: BMI085, BMI085:BMI085
- removed IC6: IIS2MDCTR, IIS2MDCTR:IIS2MDCTR
- removed J1: USB4160-03-0230-C, USB4160-03-0230-C:USB4160-03-0230-C
- removed U1: 4525DO-DS5AI001DP, 4525DO-DS5AI001DP:4525DO-DS5AI001DP
- added AIRSPEED: 4525DO-DS5AI001DP, 4525DO-DS5AI001DP:4525DO-DS5AI001DP
- added BAROMETER: DPS310XTSA1, DPS310XTSA1:DPS310XTSA1
- added C14, C15, C16, C17, C18, C23: 0.1uF, SparkFun-Capacitors:0.1UF-0603-25V-5%
- added C19, C20, C21: 1.0uF, SparkFun-Capacitors:1.0UF-0805-25V-10%
- added C22, C24, C25, C26, C27: 4.7uF, SparkFun-Capacitors:4.7UF0603
- added C28, C29: 0.1uF, SparkFun-Capacitors:0.1UF-0402-16V-10%
- added GPS: SAM-M8Q-0-10, SAM-M8Q-0-10:SAM-M8Q-0-10
- added IMU: BMI085, BMI085:BMI085
- added JP1: (no value), pinhead:PINHD-1X7
- added JP2: (no value), pinhead:PINHD-1X6
- added JP3: (no value), pinhead:PINHD-1X2
- added JP4: (no value), pinhead:PINHD-1X3
- added JP6: (no value), pinhead:PINHD-1X1
- added JP7: (no value), pinhead:PINHD-2X3
- added JST_CONNECTION: B4B-XH-A_LF__SN_, B4B-XH-A_LF__SN_:B4B-XH-A_LF__SN_
- added L1, L2, L3, L4, L5, L6, L7, L8: BLM03AG601SN1D, BLM03AG601SN1D:BLM03AG601SN1D
- added MAGNETOMETER: IIS2MDCTR, IIS2MDCTR:IIS2MDCTR
- added POWER_MODULE: LD39050PU33R, ce-capstone:LD39050PU33R
- added R10: 0, SparkFun-Resistors:0OHM-0603-1/10W-5%
- added R11, R12, R13, R14, R16, R17, R18: 22, SparkFun-Resistors:22OHM-0402-1/10W-1%
- added R6, R7, R8, R9: 4.7k, SparkFun-Resistors:4.7KOHM-0603-1/10W-1%
- added S1, S2: LL3301FF065QJ, ce-capstone:LL3301FF065QJ
- added USB_COMM_MODE_FILTER: ECMF02-4CMX8, ECMF02-4CMX8:ECMF02-4CMX8
- added Y1: ECS-TXO-3225MV-400-TR, SamacSys_Parts:ECS-TXO-3225MV-400-TR
- C3: SPICEPREFIX (none) -> C
- R4, R5: value 1.5k -> 10k; device SparkFun-Resistors:1.5KOHM-0603-1/10W-1% -> SparkFun-Resistors:10KOHM-0603-1/10W-1%
- U2: value LD39050PU33R -> TPD6F003DQDR; device ce-capstone:LD39050PU33R -> TPD6F003DQDR:TPD6F003DQDR
- renumbered IC2 to MICROCONTROLLER
Connections:
- removed net USB_DM: MICROCONTROLLER.PA11
- new net BOOT0: MICROCONTROLLER.PH3-BOOT0, R5.1, S1.3, S1.4
- new net CSB_ACCEL: IMU.CSB1, R12.2
- new net CSB_GYRO: IMU.CSB2, R13.2
- new net DN: JST_CONNECTION.3, USB_COMM_MODE_FILTER.D-_2
- new net DP: JST_CONNECTION.2, USB_COMM_MODE_FILTER.D+_2
- new net EXTI0: IMU.INT1, R14.2
- new net EXTI2: IMU.INT3, R16.2
- new net EXTI3: AIRSPEED.INT_(I2C)_/_SS_(SPI), R17.2
- new net EXTI4: MAGNETOMETER.INT/DRDY, R18.2
- new net GPS_SAFEBOOT: GPS.SAFEBOOT_N, JP6.1
- new net IMU_INT2: IMU.INT2, R10.2
- new net IMU_INT4: IMU.INT4, R10.1
- new net N$4: MICROCONTROLLER.PC8, R13.1
- new net N$8: C24.1, C4.1, IMU.VDD, L3.1
- new net N$9: C25.2, C28.2, GPS.VCC, L6.1
- new net NRST: C23.1, GPS.RESET_N, MICROCONTROLLER.NRST, POWER_MODULE.PG, R4.1, S2.1, S2.2, U2.CH4_IN
- new net NRST_O: JP7.6, U2.CH4_OUT
- new net OSC_IN: MICROCONTROLLER.PH0-OSC_IN, R11.2
- new net RX: GPS.RXD, L5.2
- new net RX_O: JP7.4, U2.CH5_OUT
- new net SWCLK: MICROCONTROLLER.PA14, U2.CH2_IN
- new net SWCLK_O: JP7.3, U2.CH2_OUT
- new net SWDIO: MICROCONTROLLER.PA13, U2.CH3_IN
- new net SWDIO_O: JP7.5, U2.CH3_OUT
- new net SWO: MICROCONTROLLER.PB3, U2.CH1_IN
- new net SWO_O: JP7.1, U2.CH1_OUT
- new net TX_O: JP7.2, U2.CH6_OUT
- new net VREF: C14.1, C19.2, L1.2, MICROCONTROLLER.VDDA/VREF+
- net 3V3: now also AIRSPEED.VCC, BAROMETER.CSB, BAROMETER.SDO, BAROMETER.VDDIO, C10.1, C15.1, C16.1, C17.1, C18.1, C20.1, C21.1, C22.1, C29.2, GPS.VCC_IO, GPS.V_BCKP, IMU.VDDIO, JP2.1, L1.1, L3.2, L6.2, L7.1, L8.2, MAGNETOMETER.CS, MAGNETOMETER.VDD_IO, MICROCONTROLLER.VDDUSB, MICROCONTROLLER.VDD_1, MICROCONTROLLER.VDD_2, MICROCONTROLLER.VDD_3, POWER_MODULE.VOUT, R4.2, R6.2, R7.1, R8.2, R9.1, S1.1, S1.2, USB_COMM_MODE_FILTER.VBUS, Y1.VDD; no longer C1.1, C11.1, C12.1, C4.1, IC1.VCC, IC1.VCC_IO, IC3.VDD, IC3.VDDIO, IC5.VDD, IC5.VDDIO, IC6.VDD, U1.VCC, U2.VOUT
- net 5V: now also JP1.1, POWER_MODULE.EN, POWER_MODULE.VIN; no longer J1.VBUS_1, J1.VBUS_2, J1.VBUS_3, J1.VBUS_4, U2.EN, U2.VIN
- net 5V_IN: now also JST_CONNECTION.4
- net GND: now also AIRSPEED.GROUND, BAROMETER.GND_1, BAROMETER.GND_2, C14.2, C15.2, C16.2, C17.2, C18.2, C19.1, C20.2, C21.2, C22.2, C23.2, C24.2, C25.1, C26.2, C27.2, C28.1, C29.1, GPS.GND_1, GPS.GND_2, GPS.GND_3, GPS.GND_4, GPS.GND_5, GPS.GND_6, GPS.GND_7, GPS.GND_8, GPS.GND_9, IMU.GNDA, IMU.GNDIO, IMU.PS, JP1.2, JP2.2, JST_CONNECTION.1, MAGNETOMETER.GND_1, MAGNETOMETER.GND_2, MICROCONTROLLER.VSSA/VREF-, MICROCONTROLLER.VSS_1, MICROCONTROLLER.VSS_2, MICROCONTROLLER.VSS_3, MICROCONTROLLER.VSS_4, POWER_MODULE.GND, R5.2, S2.3, S2.4, U2.EPAD, USB_COMM_MODE_FILTER.GND, USB_COMM_MODE_FILTER.GND_2, Y1.GROUND; no longer IC1.GND_1, IC1.GND_2, IC1.GND_3, IC1.GND_4, IC1.GND_5, IC1.GND_6, IC1.GND_7, IC1.GND_8, IC1.GND_9, IC3.GND_1, IC3.GND_2, IC5.GNDA, IC6.CS, IC6.GND_1, IC6.GND_2, J1.GND_1, J1.GND_2, J1.GND_3, J1.GND_4, J1.MH1, J1.MH2, J1.MH3, J1.MH4, R4.1, R5.1, U1.GROUND, U2.GND
- net GPIO_EXTI0: now also R14.1
- net GPIO_EXTI1: now also L4.1
- net GPIO_EXTI2: now also MICROCONTROLLER.PB2, R16.1; no longer MICROCONTROLLER.PA2
- net GPIO_EXTI3: now also MICROCONTROLLER.PC3, R17.1; no longer MICROCONTROLLER.PA3
- net GPIO_EXTI4: now also R18.1; no longer IC6.INT/DRDY
- net I2C1_SCL: now also JP2.6, MAGNETOMETER.SCL/SPC, R8.1; no longer IC6.SCL/SPC
- net I2C1_SDA: now also JP2.5, MAGNETOMETER.SDA/SDI/SDO, R9.2; no longer IC6.SDA/SDI/SDO
- net I2C2_SCL: now also BAROMETER.SCK, JP1.4; no longer IC3.SCK
- net I2C2_SDA: now also BAROMETER.SDI, JP1.3; no longer IC3.SDI
- net I2C3_SCL: now also AIRSPEED.SCL_(I2C)_/_SCLK_(SPI), JP2.4, R6.1; no longer U1.SCL_(I2C)_/_SCLK_(SPI)
- net I2C3_SDA: now also AIRSPEED.SDA_(I2C)_/_MISO_(SPI), JP2.3, R7.2; no longer U1.SDA_(I2C)_/_MISO_(SPI)
- net N$1: now also R11.1, Y1.OUTPUT; no longer IC5.GNDIO
- net N$10: now also C11.1, C12.1, C27.1, L8.1, MAGNETOMETER.VDD; no longer J1.CC2, R4.2
- net N$2: now also GPS.TIMEPULSE, L4.2; no longer FB2.1, IC1.RXD
- net N$3: now also MICROCONTROLLER.PC9, R12.1; no longer J1.CC1, R5.2
- net N$6: now also BAROMETER.VDD, C1.1, C26.1, L7.2; no longer C10.1, IC6.VDD_IO
- net N$7: now also MAGNETOMETER.C1; no longer IC6.C1
- net SPI1_MISO: now also IMU.SDO1, IMU.SDO2, JP1.6; no longer IC5.SDO1, IC5.SDO2
- net SPI1_MOSI: now also IMU.SDA/SDI, JP1.5; no longer IC5.SDA/SDI
- net SPI1_SCK: now also IMU.SCL/SCK, JP1.7; no longer IC5.SCL/SCK
- net SPI2_MISO: now also JP4.2
- net SPI2_MOSI: now also JP4.1
- net SPI2_SCK: now also JP4.3
- net TX: now also GPS.TXD, L2.2; no longer FB1.1, IC1.TXD
- net USART1_RX: now also U2.CH5_IN; no longer FB1.2
- net USART1_TX: now also U2.CH6_IN; no longer FB2.2
- net USART3_RX: now also JP3.1, L5.1
- net USART3_TX: now also JP3.2, L2.1
- net USB_DN: now also MICROCONTROLLER.PA11, USB_COMM_MODE_FILTER.D-; no longer J1.DN1, J1.DN2
- net USB_DP: now also USB_COMM_MODE_FILTER.D+; no longer J1.DP1, J1.DP2
Other:
- moved on the sheet: C1, C10, C11, C12, C13, C2, C3, C4, C5, C6, C7, C8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

Commit message: Jesus - JLC DRC updates and .GBR/BOM/CPL files
Parts:
- removed U2: TPD6F003DQDR, TPD6F003DQDR:TPD6F003DQDR
- added U1: TPD4F003DQDR, TPD4F003DQDR:TPD4F003DQDR
Connections:
- removed net RX_O: JP7.4, U2.CH5_OUT
- removed net TX_O: JP7.2, U2.CH6_OUT
- net GND: now also U1.EPAD; no longer U2.EPAD
- net NRST: now also U1.CH4_IN; no longer U2.CH4_IN
- net NRST_O: now also U1.CH4_OUT; no longer U2.CH4_OUT
- net SWCLK: now also U1.CH2_IN; no longer U2.CH2_IN
- net SWCLK_O: now also U1.CH2_OUT; no longer U2.CH2_OUT
- net SWDIO: now also U1.CH3_IN; no longer U2.CH3_IN
- net SWDIO_O: now also U1.CH3_OUT; no longer U2.CH3_OUT
- net SWO: now also U1.CH1_IN; no longer U2.CH1_IN
- net SWO_O: now also U1.CH1_OUT; no longer U2.CH1_OUT
- net USART1_RX: now also JP7.4; no longer U2.CH5_IN
- net USART1_TX: now also JP7.2; no longer U2.CH6_IN
Changed lines of the file:
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@@
 <part name="GND18" library="supply1" library_urn="urn:adsk.eagle:library:371" deviceset="GND" device=""/>
 <part name="R10" library="SparkFun-Resistors" library_urn="urn:adsk.eagle:library:532" deviceset="0OHM" device="-0603-1/10W-5%" package3d_urn="urn:adsk.eagle:package:39650/1" value="0"/>
-<part name="U2" library="TPD6F003DQDR" deviceset="TPD6F003DQDR" device=""/>
 <part name="GND19" library="supply1" library_urn="urn:adsk.eagle:library:371" deviceset="GND" device=""/>
 <part name="Y1" library="SamacSys_Parts" deviceset="ECS-TXO-3225MV-400-TR" device=""/>
@@
 <part name="JP3" library="pinhead" library_urn="urn:adsk.eagle:library:325" deviceset="PINHD-1X2" device="" package3d_urn="urn:adsk.eagle:package:22435/2"/>
 <part name="JP4" library="pinhead" library_urn="urn:adsk.eagle:library:325" deviceset="PINHD-1X3" device="" package3d_urn="urn:adsk.eagle:package:22458/2"/>
+<part name="U1" library="TPD4F003DQDR" deviceset="TPD4F003DQDR" device=""/>
 </parts>
 <sheets>
@@
 <attribute name="VALUE" x="27.94" y="-90.424" size="1.778" layer="96" font="vector" align="top-center"/>
 </instance>
-<instance part="U2" gate="A" x="-116.84" y="-15.24" smashed="yes">
-<attribute name="NAME" x="-86.0044" y="-6.1214" size="2.0828" layer="95" ratio="6" rot="SR0"/>
-<attribute name="VALUE" x="-86.6394" y="-8.6614" size="2.0828" layer="96" ratio="6" rot="SR0"/>
-</instance>
 <instance part="GND19" gate="1" x="-25.4" y="-12.7" smashed="yes">
 <attribute name="VALUE" x="-27.94" y="-15.24" size="1.778" layer="96"/>
@@
 <attribute name="NAME" x="173.99" y="33.655" size="1.778" layer="95"/>
 <attribute name="VALUE" x="173.99" y="20.32" size="1.778" layer="96"/>
+</instance>
+<instance part="U1" gate="A" x="-116.84" y="-15.24" smashed="yes">
+<attribute name="NAME" x="-86.0044" y="-6.1214" size="2.0828" layer="95" ratio="6" rot="SR0"/>
+<attribute name="VALUE" x="-86.6394" y="-8.6614" size="2.0828" layer="96" ratio="6" rot="SR0"/>
 </instance>
 </instances>
@@
 </segment>
 <segment>
-<wire x1="-114.3" y1="-25.4" x2="-134.62" y2="-25.4" width="0.1524" layer="91"/>
-<label x="-134.62" y="-25.4" size="1.778" layer="95"/>
-<pinref part="U2" gate="A" pin="CH5_IN"/>
+<wire x1="10.16" y1="-43.18" x2="-10.16" y2="-43.18" width="0.1524" layer="91"/>
+<label x="5.08" y="-43.18" size="1.778" layer="95"/>
+<pinref part="JP7" gate="A" pin="4"/>
 </segment>
 </net>
@@
 </segment>
 <segment>
-<pinref part="U2" gate="A" pin="EPAD"/>
 <wire x1="-48.26" y1="-15.24" x2="-33.02" y2="-15.24" width="0.1524" layer="91"/>
 <wire x1="-33.02" y1="-15.24" x2="-33.02" y2="-7.62" width="0.1524" layer="91"/>
@@
 <wire x1="-25.4" y1="-7.62" x2="-25.4" y2="-10.16" width="0.1524" layer="91"/>
 <pinref part="GND19" gate="1" pin="GND"/>
+<pinref part="U1" gate="A" pin="EPAD"/>
 </segment>
 <segment>
@@
 </segment>
 <segment>
-<wire x1="-114.3" y1="-27.94" x2="-134.62" y2="-27.94" width="0.1524" layer="91"/>
-<label x="-134.62" y="-27.94" size="1.778" layer="95"/>
-<pinref part="U2" gate="A" pin="CH6_IN"/>
+<wire x1="10.16" y1="-40.64" x2="-10.16" y2="-40.64" width="0.1524" layer="91"/>
+<label x="2.54" y="-40.64" size="1.778" layer="95"/>
+<pinref part="JP7" gate="A" pin="2"/>
 </segment>
 </net>
@@
 <wire x1="-114.3" y1="-22.86" x2="-134.62" y2="-22.86" width="0.1524" layer="91"/>
 <label x="-134.62" y="-22.86" size="1.778" layer="95"/>
-<pinref part="U2" gate="A" pin="CH4_IN"/>
+<pinref part="U1" gate="A" pin="CH4_IN"/>
 </segment>
 <segment>
@@
 <wire x1="-114.3" y1="-15.24" x2="-134.62" y2="-15.24" width="0.1524" layer="91"/>
 <label x="-134.62" y="-15.24" size="1.778" layer="95"/>
-<pinref part="U2" gate="A" pin="CH1_IN"/>
+<pinref part="U1" gate="A" pin="CH1_IN"/>
 </segment>
 </net>
@@
 <wire x1="-114.3" y1="-20.32" x2="-134.62" y2="-20.32" width="0.1524" layer="91"/>
 <label x="-134.62" y="-20.32" size="1.778" layer="95"/>
-<pinref part="U2" gate="A" pin="CH3_IN"/>
+<pinref part="U1" gate="A" pin="CH3_IN"/>
 </segment>
 </net>
@@
 <wire x1="-114.3" y1="-17.78" x2="-134.62" y2="-17.78" width="0.1524" layer="91"/>
 <label x="-134.62" y="-17.78" size="1.778" layer="95"/>
-<pinref part="U2" gate="A" pin="CH2_IN"/>
+<pinref part="U1" gate="A" pin="CH2_IN"/>
 </segment>
 </net>
 <net name="SWO_O" class="0">
 <segment>
-<pinref part="U2" gate="A" pin="CH1_OUT"/>
 <wire x1="-48.26" y1="-17.78" x2="-15.24" y2="-17.78" width="0.1524" layer="91"/>
 <label x="-38.1" y="-17.78" size="1.778" layer="95"/>
+<pinref part="U1" gate="A" pin="CH1_OUT"/>
 </segment>
 <segment>
@@
 <net name="SWCLK_O" class="0">
 <segment>
-<pinref part="U2" gate="A" pin="CH2_OUT"/>
 <wire x1="-48.26" y1="-20.32" x2="-15.24" y2="-20.32" width="0.1524" layer="91"/>
 <label x="-38.1" y="-20.32" size="1.778" layer="95"/>
+<pinref part="U1" gate="A" pin="CH2_OUT"/>
 </segment>
 <segment>
@@
 <net name="SWDIO_O" class="0">
 <segment>
-<pinref part="U2" gate="A" pin="CH3_OUT"/>
 <wire x1="-48.26" y1="-22.86" x2="-15.24" y2="-22.86" width="0.1524" layer="91"/>
 <label x="-38.1" y="-22.86" size="1.778" layer="95"/>
+<pinref part="U1" gate="A" pin="CH3_OUT"/>
 </segment>
 <segment>
@@
 <net name="NRST_O" class="0">
 <segment>
-<pinref part="U2" gate="A" pin="CH4_OUT"/>
 <wire x1="-48.26" y1="-25.4" x2="-15.24" y2="-25.4" width="0.1524" layer="91"/>
 <label x="-38.1" y="-25.4" size="1.778" layer="95"/>
+<pinref part="U1" gate="A" pin="CH4_OUT"/>
 </segment>
 <segment>
@@
 </segment>
 </net>
-<net name="RX_O" class="0">
-<segment>
-<pinref part="U2" gate="A" pin="CH5_OUT"/>
-<wire x1="-48.26" y1="-27.94" x2="-15.24" y2="-27.94" width="0.1524" layer="91"/>
-<label x="-38.1" y="-27.94" size="1.778" layer="95"/>
-</segment>
-<segment>
-<pinref part="JP7" gate="A" pin="4"/>
-<wire x1="-10.16" y1="-43.18" x2="2.54" y2="-43.18" width="0.1524" layer="91"/>
-<label x="0" y="-43.18" size="1.778" layer="95"/>
-</segment>
-</net>
-<net name="TX_O" class="0">
-<segment>
-<pinref part="U2" gate="A" pin="CH6_OUT"/>
-<wire x1="-48.26" y1="-30.48" x2="-15.24" y2="-30.48" width="0.1524" layer="91"/>
-<label x="-38.1" y="-30.48" size="1.778" layer="95"/>
-</segment>
-<segment>
-<pinref part="JP7" gate="A" pin="2"/>
-<wire x1="-10.16" y1="-40.64" x2="2.54" y2="-40.64" width="0.1524" layer="91"/>
-<label x="0" y="-40.64" size="1.778" layer="95"/>
-</segment>
-</net>
