File: PCB_Sensor_Stick/SensorStick_IMUedits_HeaderPins_jesus.brd (EAGLE design)
At the start: 63.5 x 38.1 mm, 53 parts, among them U1 ECMF02-4CMX8, U2 TPD6F003DQDR

Commit message: J - Current version with various changes according the feedback
Parts:
- added C23: 0.1uF, SparkFun-Capacitors:0603
- added C24, C25, C26: 1.0uF, SparkFun-Capacitors:0402
- added R4: 10k, SparkFun-Resistors:0603
- added S2: LL3301FF065QJ, ce-capstone:LL3301FF065QJ
- added USB_COMM_MODE_FILTER: ECMF02-4CMX8, ECMF02-4CMX8:MICRO_QFN-8L_STM
- added Y1: ECS-TXO-3225MV-400-TR, SamacSys_Parts:ECSTXO3225MV400TR
- U1: value ECMF02-4CMX8 -> LT1461CIS8-3PBF; device ECMF02-4CMX8:MICRO_QFN-8L_STM -> LT1461:SO-8_S_LIT
- moved U1 44.2 mm to (-14.7, -55.6)
- moved R10 15.9 mm to (-14.5, 12.2)
Connections:
- new net GPS_MEM: GPS.8
- new net N$1: MICROCONTROLLER.5
- new net N$10: AIRSPEED.2, C25.1, C26.1, C3.2, U1.6
- new net N$3: MICROCONTROLLER.6
- new net N$4: Y1.3
- new net N$6: C24.1, U1.2
- net 3V3: now also R4.2, USB_COMM_MODE_FILTER.1, Y1.4; no longer AIRSPEED.2, C3.2, U1.1
- net DN: now also USB_COMM_MODE_FILTER.2; no longer U1.2
- net DP: now also USB_COMM_MODE_FILTER.3; no longer U1.3
- net GND: now also C23.2, C24.2, C25.2, C26.2, S2.3, S2.4, U1.4, USB_COMM_MODE_FILTER.5, USB_COMM_MODE_FILTER.8, Y1.2; no longer U1.5, U1.8
- net GPIO_EXTI0: no longer JP2.3
- net GPIO_EXTI4: now also JP2.3
- net NRST: now also C23.1, R4.1, S2.1, S2.2
- net USB_DN: now also USB_COMM_MODE_FILTER.7; no longer U1.7
- net USB_DP: now also USB_COMM_MODE_FILTER.6; no longer U1.6
Routing:
- net 3V3: track 108.4 -> 105.0 mm, vias 21 -> 20

Commit message: Jesus - Edits to PCB schematic/layout
Parts:
- removed FB1, FB2: BLM15HD102SN1, BLM15HD102SN1:NFZ15SG152SN10B
- removed U1: LT1461CIS8-3PBF, LT1461:SO-8_S_LIT
- added C27: 4.7uF, SparkFun-Capacitors:0603
- added C28, C29: 0.1uF, SparkFun-Capacitors:0402
- added JP7: (no value), pinhead:2X03
- added L2, L3, L4, L5, L6, L7, L8: BLM03AG601SN1D, BLM03AG601SN1D:IND_BLM03_0201_MUR
- added R11, R12, R13, R14, R16, R17, R18: 22, SparkFun-Resistors:0402
- C24, C25, C26: value 1.0uF -> 4.7uF; device SparkFun-Capacitors:0402 -> SparkFun-Capacitors:0603
- JP6: device pinhead:1X06 -> pinhead:1X01
- L1: value (none) -> BLM03AG601SN1D; device rcl:L4035M -> BLM03AG601SN1D:IND_BLM03_0201_MUR
- moved C24 147.0 mm to (94.2, 5.08)
- moved C25 147.0 mm to (94.2, 1.78)
- moved C26 147.0 mm to (94.2, -1.52)
- moved R4 131.8 mm to (57.9, 15.0)
- moved C23 106.6 mm to (60.2, 10.2), turned to 270 degrees
- moved S2 103.3 mm to (68.1, 4.57)
- moved R10 79.2 mm to (63.0, 28.4), turned to 90 degrees
- moved Y1 78.7 mm to (53.3, 16.8), turned to 90 degrees
- moved JP6 48.3 mm to (23.6, 3.56)
- moved USB_COMM_MODE_FILTER 46.8 mm to (14.2, 26.4), turned to 270 degrees
- moved S1 45.0 mm to (45.0, 6.35), turned to 180 degrees
- moved R5 39.3 mm to (38.6, 4.83), turned to 270 degrees
- moved JP2 34.2 mm to (67.3, 45.2), turned to 0 degrees
- moved JP4 30.5 mm to (46.7, 45.5), turned to 0 degrees
- moved JP5 26.5 mm to (84.3, 27.7), turned to 270 degrees
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Connections:
- removed net GPS_MEM: GPS.8
- new net EXTI0: IMU.16, R14.2
- new net EXTI2: IMU.12, R16.2
- new net EXTI3: AIRSPEED.5, R17.2
- new net EXTI4: MAGNETOMETER.7, R18.2
- new net GPS_SAFEBOOT: GPS.8, JP6.1
- new net IMU_INT2: IMU.1, R10.2
- new net IMU_INT4: IMU.13, R10.1
- new net N$8: C24.1, C4.1, IMU.3, L3.1
- new net N$9: C25.2, C28.2, GPS.17, L6.1
- new net OSC_IN: MICROCONTROLLER.5, R11.2
- new net RX: GPS.14, L5.2
- net 3V3: now also AIRSPEED.2, C29.2, C3.2, L1.1, L3.2, L6.2, L7.1, L8.2; no longer BAROMETER.8, C1.1, C11.1, C12.1, C4.1, GPS.17, IMU.3, L1.2, MAGNETOMETER.9
- net CSB_ACCEL: now also R12.2; no longer MICROCONTROLLER.39
- net CSB_GYRO: now also R13.2; no longer MICROCONTROLLER.40
- net GND: now also C25.1, C27.2, C28.1, C29.1; no longer C24.2, C25.2, U1.4
- net GPIO_EXTI0: now also R14.1; no longer IMU.16
- net GPIO_EXTI1: now also L4.1; no longer AIRSPEED.5
- net GPIO_EXTI2: now also MICROCONTROLLER.28, R16.1; no longer IMU.12, MICROCONTROLLER.16, R10.1
- net GPIO_EXTI3: now also MICROCONTROLLER.11, R17.1; no longer MAGNETOMETER.7, MICROCONTROLLER.17
- net GPIO_EXTI4: now also R18.1; no longer IMU.1, R10.2
- net N$1: now also R11.1, Y1.3; no longer MICROCONTROLLER.5
- net N$10: now also C11.1, C12.1, C27.1, L8.1, MAGNETOMETER.9; no longer AIRSPEED.2, C25.1, C26.1, C3.2, U1.6
- net N$2: now also GPS.7, L4.2; no longer FB2.1, GPS.14
- net N$3: now also MICROCONTROLLER.40, R12.1; no longer MICROCONTROLLER.6
- net N$4: now also MICROCONTROLLER.39, R13.1; no longer Y1.3
- net N$6: now also BAROMETER.8, C1.1, C26.1, L7.2; no longer C24.1, U1.2
- net NRST_O: now also JP7.6; no longer JP6.4
- net RX_O: now also JP7.4; no longer JP6.5
- net SWCLK_O: now also JP7.3; no longer JP6.2
- net SWDIO_O: now also JP7.5; no longer JP6.3
- net SWO_O: now also JP7.1; no longer JP6.1
- net TX: now also L2.2; no longer FB1.1
- net TX_O: now also JP7.2; no longer JP6.6
- net USART1_RX: now also U2.5; no longer FB1.2
- net USART1_TX: now also U2.6; no longer FB2.2
- net USART3_RX: now also L5.1; no longer U2.5
- net USART3_TX: now also L2.1; no longer U2.6
- net VREF: now also L1.2; no longer L1.1
Routing:
- net NRST: track 0.00 -> 112.8 mm, vias 0 -> 4
- net GPIO_EXTI0: track 58.4 -> 19.8 mm, vias 3 -> 2
- net GPIO_EXTI2: track 40.1 -> 10.4 mm, vias 3 -> 0
- net CSB_GYRO: track 38.4 -> 8.81 mm
- net N$4: track 0.00 -> 28.3 mm, vias 0 -> 2
- net GPIO_EXTI1: track 30.5 -> 55.8 mm, vias 2 -> 4
- net I2C2_SCL: track 34.7 -> 10.0 mm, vias 2 -> 0
- net N$3: track 0.00 -> 24.2 mm, vias 0 -> 2
- net SWDIO: track 0.00 -> 23.3 mm, vias 0 -> 2
- net GND: track 178.9 -> 155.8 mm, vias 27 -> 34
- net EXTI0: track 0.00 -> 21.3 mm, vias 0 -> 2
- net USART3_TX: track 0.00 -> 21.0 mm, vias 0 -> 2
- net BOOT0: track 0.00 -> 20.3 mm
- net IMU_INT4: track 0.00 -> 19.8 mm, vias 0 -> 2
- net I2C2_SDA: track 30.1 -> 10.6 mm, vias 3 -> 2
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Other:
- board size 63.5 x 38.1 mm -> 76.2 x 44.5 mm
