File: PCB_Sensor_Stick/SensorStick_IMUedits_HeaderPins_jesus.sch (EAGLE design)
At the start: 61 parts, among them U1 LT1461CIS8-3PBF, U2 TPD6F003DQDR, Y1 ECS-TXO-3225MV-400-TR

Commit message: Jesus - Edits to PCB schematic/layout
Parts:
- removed FB1, FB2: BLM15HD102SN1, BLM15HD102SN1:BLM15HD102SN1
- removed U1: LT1461CIS8-3PBF, LT1461:LT1461CIS8-3PBF
- added C27: 4.7uF, SparkFun-Capacitors:4.7UF0603
- added C28, C29: 0.1uF, SparkFun-Capacitors:0.1UF-0402-16V-10%
- added JP7: (no value), pinhead:PINHD-2X3
- added L2, L3, L4, L5, L6, L7, L8: BLM03AG601SN1D, BLM03AG601SN1D:BLM03AG601SN1D
- added R11, R12, R13, R14, R16, R17, R18: 22, SparkFun-Resistors:22OHM-0402-1/10W-1%
- C24, C25, C26: value 1.0uF -> 4.7uF; device SparkFun-Capacitors:1.0UF-0402-16V-10% -> SparkFun-Capacitors:4.7UF0603
- JP6: device pinhead:PINHD-1X6 -> pinhead:PINHD-1X1
- L1: value (none) -> BLM03AG601SN1D; device rcl:L-USL4035M -> BLM03AG601SN1D:BLM03AG601SN1D
Connections:
- removed net GPS_MEM: GPS.SAFEBOOT_N
- new net EXTI0: IMU.INT1, R14.2
- new net EXTI2: IMU.INT3, R16.2
- new net EXTI3: AIRSPEED.INT_(I2C)_/_SS_(SPI), R17.2
- new net EXTI4: MAGNETOMETER.INT/DRDY, R18.2
- new net GPS_SAFEBOOT: GPS.SAFEBOOT_N, JP6.1
- new net IMU_INT2: IMU.INT2, R10.2
- new net IMU_INT4: IMU.INT4, R10.1
- new net N$8: C24.1, C4.1, IMU.VDD, L3.1
- new net N$9: C25.2, C28.2, GPS.VCC, L6.1
- new net OSC_IN: MICROCONTROLLER.PH0-OSC_IN, R11.2
- new net RX: GPS.RXD, L5.2
- net 3V3: now also AIRSPEED.VCC, C29.2, C3.2, L1.1, L3.2, L6.2, L7.1, L8.2; no longer BAROMETER.VDD, C1.1, C11.1, C12.1, C4.1, GPS.VCC, IMU.VDD, L1.2, MAGNETOMETER.VDD
- net CSB_ACCEL: now also R12.2; no longer MICROCONTROLLER.PC8
- net CSB_GYRO: now also R13.2; no longer MICROCONTROLLER.PC9
- net GND: now also C25.1, C27.2, C28.1, C29.1; no longer C24.2, C25.2, U1.GND
- net GPIO_EXTI0: now also R14.1; no longer IMU.INT1
- net GPIO_EXTI1: now also L4.1; no longer AIRSPEED.INT_(I2C)_/_SS_(SPI)
- net GPIO_EXTI2: now also MICROCONTROLLER.PB2, R16.1; no longer IMU.INT3, MICROCONTROLLER.PA2, R10.1
- net GPIO_EXTI3: now also MICROCONTROLLER.PC3, R17.1; no longer MAGNETOMETER.INT/DRDY, MICROCONTROLLER.PA3
- net GPIO_EXTI4: now also R18.1; no longer IMU.INT2, R10.2
- net N$1: now also R11.1, Y1.OUTPUT; no longer MICROCONTROLLER.PH0-OSC_IN
- net N$10: now also C11.1, C12.1, C27.1, L8.1, MAGNETOMETER.VDD; no longer AIRSPEED.VCC, C25.1, C26.1, C3.2, U1.VOUT
- net N$2: now also GPS.TIMEPULSE, L4.2; no longer FB2.1, GPS.RXD
- net N$3: now also MICROCONTROLLER.PC9, R12.1; no longer MICROCONTROLLER.PH1-OSC_OUT
- net N$4: now also MICROCONTROLLER.PC8, R13.1; no longer Y1.OUTPUT
- net N$6: now also BAROMETER.VDD, C1.1, C26.1, L7.2; no longer C24.1, U1.VIN
- net NRST_O: now also JP7.6; no longer JP6.4
- net RX_O: now also JP7.4; no longer JP6.5
- net SWCLK_O: now also JP7.3; no longer JP6.2
- net SWDIO_O: now also JP7.5; no longer JP6.3
- net SWO_O: now also JP7.1; no longer JP6.1
- net TX: now also L2.2; no longer FB1.1
- net TX_O: now also JP7.2; no longer JP6.6
- net USART1_RX: now also U2.CH5_IN; no longer FB1.2
- net USART1_TX: now also U2.CH6_IN; no longer FB2.2
- net USART3_RX: now also L5.1; no longer U2.CH5_IN
- net USART3_TX: now also L2.1; no longer U2.CH6_IN
- net VREF: now also L1.2; no longer L1.1
Other:
- moved on the sheet: BAROMETER, C1, C10, C11, C12, C13, C14, C15, C16, C17, C18, C19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
