File: PCB_Sensor_Stick/SensorStick.brd (EAGLE design)
At the start: 76.2 x 44.5 mm, 75 parts, among them U2 TPD6F003DQDR, Y1 ECS-TXO-3225MV-400-TR

Commit message: Jesus - JLC DRC updates and .GBR/BOM/CPL files
Parts:
- removed U2: TPD6F003DQDR, TPD6F003DQDR:DQD12_2X0P4
- added U1: TPD4F003DQDR, TPD4F003DQDR:DQD8_1P2X0P4
- moved C24 0.25 mm to (64.3, 34.3)
- moved C22 0.25 mm to (33.5, 31.1)
- moved C4 0.25 mm to (62.6, 35.2)
- moved L3 0.25 mm to (55.1, 39.9)
Connections:
- removed net RX_O: JP7.4, U2.8
- removed net TX_O: JP7.2, U2.7
- net GND: now also U1.9; no longer U2.13
- net NRST: now also U1.4; no longer U2.4
- net NRST_O: now also U1.5; no longer U2.9
- net SWCLK: now also U1.2; no longer U2.2
- net SWCLK_O: now also U1.7; no longer U2.11
- net SWDIO: now also U1.3; no longer U2.3
- net SWDIO_O: now also U1.6; no longer U2.10
- net SWO: now also U1.1; no longer U2.1
- net SWO_O: now also U1.8; no longer U2.12
- net USART1_RX: now also JP7.4; no longer U2.5
- net USART1_TX: now also JP7.2; no longer U2.6
Routing:
- net TX_O: track 17.7 -> 0.00 mm
- net USART1_TX: track 14.2 -> 30.5 mm
- net USART1_RX: track 13.4 -> 27.6 mm
- net RX_O: track 13.7 -> 0.00 mm
- net N$8: track 17.0 -> 18.0 mm
- net SWO: track 14.4 -> 13.5 mm
- net SWDIO: track 23.3 -> 22.5 mm
- net IMU_INT2: track 14.3 -> 15.1 mm
- net SWCLK: track 14.5 -> 13.8 mm
- net N$3: track 24.2 -> 23.5 mm
- net NRST_O: track 8.09 -> 8.65 mm
Other:
- board text added: "JST"
- board text added: "MAG"
- board text added: "PWR"
- board text added: "Project Dragonfly UCSB Capstone"
