File: PCB/v1/SensorStick.brd (EAGLE design)
At the start: 76.2 x 44.5 mm, 75 parts, among them U1 TPD4F003DQDR, Y1 ECS-TXO-3225MV-400-TR

Commit message: Jesus - Edits to v1 for 2nd print
Parts:
- removed R4: 10k, SparkFun-Resistors:0603
Connections:
- net 3V3: now also Y1.1; no longer R4.2
- net NRST: no longer R4.1
Routing:
- net NRST: track 118.6 -> 115.0 mm
- net 3V3: track 144.8 -> 146.6 mm
- net GND: track 178.5 -> 180.0 mm
Changed lines of the file:
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@@
 <attribute name="VALUE" x="59.182" y="12.7" size="0.6096" layer="27" font="vector" ratio="20" rot="R270" align="top-center"/>
-</element>
-<element name="R4" library="SparkFun-Resistors" library_urn="urn:adsk.eagle:library:532" package="0603" package3d_urn="urn:adsk.eagle:package:39650/1" value="10k" x="57.658" y="17.526" smashed="yes">
-<attribute name="NAME" x="57.658" y="18.288" size="0.6096" layer="25" font="vector" ratio="20" align="bottom-center"/>
-<attribute name="PROD_ID" value="RES-00824" x="57.658" y="17.526" size="1.778" layer="27" display="off"/>
-<attribute name="VALUE" x="57.658" y="16.764" size="0.6096" layer="27" font="vector" ratio="20" align="top-center"/>
 </element>
 <element name="L2" library="BLM03AG601SN1D" package="IND_BLM03_0201_MUR" value="BLM03AG601SN1D" x="22.352" y="12.446" smashed="yes" rot="R180">
@@
 <contactref element="USB_COMM_MODE_FILTER" pad="1"/>
 <contactref element="Y1" pad="4"/>
-<contactref element="R4" pad="2"/>
 <contactref element="C3" pad="2"/>
 <contactref element="AIRSPEED" pad="2"/>
@@
 <wire x1="54.86" y1="3.552" x2="54.61" y2="3.302" width="0.2032" layer="1"/>
 <via x="54.61" y="3.302" extent="1-16" drill="0.35"/>
-<wire x1="58.508" y1="17.526" x2="58.508" y2="18.2" width="0.2032" layer="1"/>
-<wire x1="58.508" y1="18.2" x2="57.912" y2="18.796" width="0.2032" layer="1"/>
 <via x="57.912" y="18.796" extent="1-16" drill="0.35"/>
 <wire x1="57.912" y1="20.232" x2="57.912" y2="18.796" width="0.2032" layer="1"/>
@@
 <wire x1="37.652" y1="31.519" x2="37.652" y2="32.70083125" width="0.2032" layer="1"/>
 <wire x1="37.652" y1="32.70083125" x2="37.33283125" y2="33.02" width="0.2032" layer="1"/>
+<contactref element="Y1" pad="1"/>
+<wire x1="52.324" y1="16.256" x2="53.594" y2="16.256" width="0.1524" layer="1"/>
+<wire x1="53.594" y1="16.256" x2="54.036" y2="16.698" width="0.1524" layer="1"/>
+<wire x1="54.036" y1="16.698" x2="54.036" y2="18.154" width="0.1524" layer="1"/>
 </signal>
 <signal name="USART1_RX">
@@
 <wire x1="34.544" y1="39.624" x2="34.888" y2="39.28" width="0.2032" layer="1"/>
 <wire x1="34.888" y1="39.28" x2="34.888" y2="38.313" width="0.2032" layer="1"/>
-<wire x1="24.638" y1="36.703" x2="24.638" y2="35.052" width="0.3048" layer="1"/>
-<wire x1="24.638" y1="35.052" x2="23.876" y2="34.29" width="0.3048" layer="1"/>
+<wire x1="24.638" y1="36.703" x2="24.13" y2="36.195" width="0.3048" layer="1"/>
+<wire x1="24.13" y1="36.195" x2="24.13" y2="34.544" width="0.3048" layer="1"/>
+<wire x1="24.13" y1="34.544" x2="23.876" y2="34.29" width="0.3048" layer="1"/>
 <wire x1="23.876" y1="34.29" x2="22.098" y2="34.29" width="0.3048" layer="1"/>
 <wire x1="22.098" y1="34.29" x2="21.844" y2="34.036" width="0.3048" layer="1"/>
@@
 <wire x1="73.866" y1="4.62" x2="73.914" y2="4.572" width="0.2032" layer="1"/>
 <via x="73.914" y="4.572" extent="1-16" drill="0.35"/>
-<wire x1="67.818" y1="2.54" x2="67.818" y2="4.318" width="0.2032" layer="1"/>
-<via x="67.818" y="4.318" extent="1-16" drill="0.35"/>
+<wire x1="67.818" y1="4.064" x2="67.31" y2="4.572" width="0.2032" layer="1"/>
+<wire x1="66.294" y1="4.572" x2="67.31" y2="4.572" width="0.2032" layer="1"/>
+<wire x1="67.818" y1="2.54" x2="67.818" y2="4.064" width="0.2032" layer="1"/>
+<via x="66.294" y="4.572" extent="1-16" drill="0.35"/>
 <wire x1="30.48" y1="36.267" x2="29.519" y2="36.267" width="0.2032" layer="1"/>
 <wire x1="29.519" y1="36.267" x2="29.21" y2="36.576" width="0.2032" layer="1"/>
@@
 <contactref element="GPS" pad="18"/>
 <contactref element="POWER_MODULE" pad="3"/>
-<contactref element="S2" pad="1"/>
-<contactref element="S2" pad="2"/>
-<contactref element="C23" pad="1"/>
-<contactref element="R4" pad="1"/>
 <wire x1="47.14" y1="25.031" x2="48.375" y2="25.031" width="0.2032" layer="1"/>
 <wire x1="49.0194" y1="24.3866" x2="49.9583" y2="24.3866" width="0.2032" layer="1"/>
 <wire x1="49.9583" y1="24.3866" x2="49.9609" y2="24.384" width="0.2032" layer="1"/>
 <wire x1="49.9609" y1="24.384" x2="54.102" y2="24.384" width="0.2032" layer="1"/>
-<wire x1="54.102" y1="24.384" x2="56.808" y2="21.678" width="0.2032" layer="1"/>
+<wire x1="54.102" y1="24.384" x2="56.944" y2="21.542" width="0.2032" layer="1"/>
 <wire x1="48.375" y1="25.031" x2="49.0194" y2="24.3866" width="0.2032" layer="1"/>
-<wire x1="56.808" y1="17.526" x2="56.944" y2="17.39" width="0.2032" layer="1"/>
-<wire x1="56.808" y1="17.526" x2="56.808" y2="21.678" width="0.2032" layer="1"/>
-<wire x1="56.944" y1="15.446" x2="56.944" y2="17.39" width="0.2032" layer="1"/>
 <wire x1="37.9758" y1="11.3058" x2="37.9758" y2="11.938" width="0.1524" layer="1"/>
 <via x="37.9758" y="11.938" extent="1-16" drill="0.35"/>
 <wire x1="37.9758" y1="11.938" x2="37.2138" y2="12.7" width="0.2032" layer="16"/>
-<wire x1="60.872" y1="13.55" x2="59.944" y2="13.55" width="0.2032" layer="1"/>
-<wire x1="67.866" y1="10.886" x2="67.866" y2="11.986" width="0.2032" layer="1"/>
-<wire x1="67.866" y1="11.986" x2="68.58" y2="12.7" width="0.2032" layer="1"/>
-<wire x1="68.58" y1="12.7" x2="72.898" y2="12.7" width="0.2032" layer="1"/>
-<wire x1="72.898" y1="12.7" x2="73.866" y2="11.732" width="0.2032" layer="1"/>
-<wire x1="73.866" y1="11.732" x2="73.866" y2="10.886" width="0.2032" layer="1"/>
-<wire x1="59.944" y1="13.55" x2="58.84" y2="13.55" width="0.2032" layer="1"/>
-<wire x1="58.84" y1="13.55" x2="57.912" y2="14.478" width="0.2032" layer="1"/>
+<wire x1="57.912" y1="14.478" x2="58.801" y2="13.589" width="0.2032" layer="1"/>
 <wire x1="57.912" y1="14.478" x2="56.944" y2="15.446" width="0.2032" layer="1"/>
 <wire x1="57.912" y1="14.478" x2="45.974" y2="14.478" width="0.2032" layer="1"/>
@@
 <wire x1="12.446" y1="22.606" x2="12.446" y2="19.173" width="0.2032" layer="1"/>
 <wire x1="12.446" y1="19.173" x2="12.319" y2="19.046" width="0.2032" layer="1"/>
-<wire x1="67.866" y1="10.886" x2="67.83" y2="10.922" width="0.2032" layer="1"/>
-<wire x1="67.83" y1="10.922" x2="61.976" y2="10.922" width="0.2032" layer="1"/>
-<wire x1="61.976" y1="10.922" x2="61.214" y2="11.684" width="0.2032" layer="1"/>
-<wire x1="61.214" y1="13.208" x2="60.872" y2="13.55" width="0.2032" layer="1"/>
-<wire x1="61.214" y1="11.684" x2="61.214" y2="13.208" width="0.2032" layer="1"/>
 <wire x1="37.2138" y1="12.7" x2="29.464" y2="12.7" width="0.2032" layer="16"/>
 <wire x1="29.464" y1="12.7" x2="27.686" y2="14.478" width="0.2032" layer="16"/>
@@
 <wire x1="36.693" y1="10.76" x2="37.43" y2="10.76" width="0.1524" layer="1"/>
 <wire x1="37.43" y1="10.76" x2="37.9758" y2="11.3058" width="0.1524" layer="1"/>
+<contactref element="C23" pad="1"/>
+<contactref element="S2" pad="1"/>
+<contactref element="S2" pad="2"/>
+<wire x1="56.944" y1="21.542" x2="56.944" y2="15.446" width="0.2032" layer="1"/>
+<wire x1="59.905" y1="13.589" x2="59.944" y2="13.55" width="0.1524" layer="1"/>
+<wire x1="73.866" y1="10.886" x2="67.866" y2="10.886" width="0.2032" layer="1"/>
+<wire x1="67.866" y1="10.886" x2="62.608" y2="10.886" width="0.2032" layer="1"/>
+<wire x1="62.608" y1="10.886" x2="59.944" y2="13.55" width="0.2032" layer="1"/>
+<wire x1="58.801" y1="13.589" x2="59.905" y2="13.589" width="0.2032" layer="1"/>
 </signal>
 <signal name="DP">
