File: PCB/v1/SensorStick.sch (EAGLE design)
At the start: 76 parts, among them U2 TPD6F003DQDR, Y1 ECS-TXO-3225MV-400-TR

Commit message: Jesus - PCB version control
Parts:
- removed JP5: (no value), pinhead:PINHD-2X3
- removed U2: TPD6F003DQDR, TPD6F003DQDR:TPD6F003DQDR
- added U1: TPD4F003DQDR, TPD4F003DQDR:TPD4F003DQDR
- JP1: device pinhead:PINHD-2X2 -> pinhead:PINHD-1X7
- JP2: device pinhead:PINHD-2X2 -> pinhead:PINHD-1X6
- JP3: device pinhead:PINHD-2X2 -> pinhead:PINHD-1X2
- JP4: device pinhead:PINHD-1X5 -> pinhead:PINHD-1X3
Connections:
- removed net N$11: JP5.6
- removed net RX_O: JP7.4, U2.CH5_OUT
- removed net TX_O: JP7.2, U2.CH6_OUT
- net 3V3: now also JP2.1; no longer JP4.1, JP5.1
- net GND: now also C24.2, JP1.2, JP2.2, U1.EPAD; no longer JP1.3, JP4.2, JP5.2, U2.EPAD
- net GPIO_EXTI2: no longer JP2.1
- net GPIO_EXTI4: no longer JP2.3
- net I2C1_SCL: now also JP2.6; no longer JP3.2
- net I2C1_SDA: now also JP2.5; no longer JP3.4
- net I2C2_SDA: now also JP1.3; no longer JP1.2
- net I2C3_SCL: now also JP2.4; no longer JP5.3
- net I2C3_SDA: now also JP2.3; no longer JP5.5
- net NRST: now also U1.CH4_IN; no longer U2.CH4_IN
- net NRST_O: now also U1.CH4_OUT; no longer U2.CH4_OUT
- net SPI1_MISO: now also JP1.6; no longer JP2.2
- net SPI1_MOSI: now also JP1.5; no longer JP2.4
- net SPI1_SCK: now also JP1.7; no longer JP5.4
- net SPI2_MISO: now also JP4.2; no longer JP4.4
- net SPI2_MOSI: now also JP4.1; no longer JP4.5
- net SWCLK: now also U1.CH2_IN; no longer U2.CH2_IN
- net SWCLK_O: now also U1.CH2_OUT; no longer U2.CH2_OUT
- net SWDIO: now also U1.CH3_IN; no longer U2.CH3_IN
- net SWDIO_O: now also U1.CH3_OUT; no longer U2.CH3_OUT
- net SWO: now also U1.CH1_IN; no longer U2.CH1_IN
- net SWO_O: now also U1.CH1_OUT; no longer U2.CH1_OUT
- net USART1_RX: now also JP7.4; no longer JP3.3, U2.CH5_IN
- net USART1_TX: now also JP7.2; no longer JP3.1, U2.CH6_IN
- net USART3_RX: now also JP3.1
- net USART3_TX: now also JP3.2
Other:
- moved on the sheet: AIRSPEED, BAROMETER, C1, C10, C11, C12, C13, C14, C15, C16, C17, C18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

Commit message: Jesus - Edits to v1 for 2nd print
Parts:
- removed R4: 10k, SparkFun-Resistors:10KOHM-0603-1/10W-1%
Connections:
- net 3V3: now also Y1.TRI-STATE; no longer R4.2
- net NRST: no longer R4.1
Changed lines of the file:
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@@
 <part name="GND20" library="supply1" library_urn="urn:adsk.eagle:library:371" deviceset="GND" device=""/>
 <part name="GND22" library="supply1" library_urn="urn:adsk.eagle:library:371" deviceset="GND" device=""/>
-<part name="R4" library="SparkFun-Resistors" library_urn="urn:adsk.eagle:library:532" deviceset="10KOHM" device="-0603-1/10W-1%" package3d_urn="urn:adsk.eagle:package:39650/1" value="10k"/>
 <part name="L2" library="BLM03AG601SN1D" deviceset="BLM03AG601SN1D" device=""/>
 <part name="L4" library="BLM03AG601SN1D" deviceset="BLM03AG601SN1D" device=""/>
@@
 <attribute name="VALUE" x="-142.24" y="129.54" size="1.778" layer="96"/>
 </instance>
-<instance part="R4" gate="G$1" x="-50.8" y="104.14" smashed="yes" rot="R90">
-<attribute name="NAME" x="-52.324" y="104.14" size="1.778" layer="95" font="vector" rot="R90" align="bottom-center"/>
-<attribute name="VALUE" x="-49.276" y="104.14" size="1.778" layer="96" font="vector" rot="R90" align="top-center"/>
-</instance>
 <instance part="L2" gate="A" x="101.6" y="-71.12" smashed="yes">
 <attribute name="VALUE" x="86.9188" y="-80.4672" size="3.4798" layer="96" ratio="10" rot="SR0"/>
@@
 </segment>
 <segment>
-<pinref part="R4" gate="G$1" pin="2"/>
-<wire x1="-50.8" y1="109.22" x2="-50.8" y2="116.84" width="0.1524" layer="91"/>
-<label x="-50.8" y="114.3" size="1.778" layer="95"/>
-</segment>
-<segment>
 <pinref part="C3" gate="G$1" pin="2"/>
 <wire x1="170.18" y1="-25.4" x2="177.8" y2="-25.4" width="0.1524" layer="91"/>
@@
 <wire x1="307.34" y1="-27.94" x2="299.72" y2="-27.94" width="0.1524" layer="91"/>
 <label x="297.18" y="-27.94" size="1.778" layer="95"/>
+</segment>
+<segment>
+<pinref part="Y1" gate="G$1" pin="TRI-STATE"/>
+<wire x1="-182.88" y1="139.7" x2="-193.04" y2="139.7" width="0.1524" layer="91"/>
+<wire x1="-193.04" y1="139.7" x2="-193.04" y2="132.08" width="0.1524" layer="91"/>
+<label x="-193.04" y="132.08" size="1.778" layer="95"/>
 </segment>
 </net>
@@
 </segment>
 <segment>
+<pinref part="C23" gate="G$1" pin="1"/>
+<wire x1="-71.12" y1="86.36" x2="-71.12" y2="93.98" width="0.1524" layer="91"/>
 <pinref part="S2" gate="G$1" pin="1"/>
+<wire x1="-71.12" y1="93.98" x2="-50.8" y2="93.98" width="0.1524" layer="91"/>
 <pinref part="S2" gate="G$1" pin="2"/>
-<wire x1="-45.72" y1="93.98" x2="-50.8" y2="93.98" width="0.1524" layer="91"/>
-<wire x1="-50.8" y1="93.98" x2="-71.12" y2="93.98" width="0.1524" layer="91"/>
+<wire x1="-50.8" y1="93.98" x2="-45.72" y2="93.98" width="0.1524" layer="91"/>
 <junction x="-50.8" y="93.98"/>
 <wire x1="-71.12" y1="93.98" x2="-78.74" y2="93.98" width="0.1524" layer="91"/>
-<wire x1="-50.8" y1="93.98" x2="-50.8" y2="99.06" width="0.1524" layer="91"/>
-<pinref part="C23" gate="G$1" pin="1"/>
-<wire x1="-71.12" y1="86.36" x2="-71.12" y2="93.98" width="0.1524" layer="91"/>
 <junction x="-71.12" y="93.98"/>
 <label x="-78.74" y="93.98" size="1.778" layer="95"/>
-<pinref part="R4" gate="G$1" pin="1"/>
-</segment>
-</net>
+</segment>
+</net>
