File: PCB/v1/v2/SensorStick_v2.sch (EAGLE design)
At the start: 58 parts, among them IC1 STM32L412RBT6, J2 10118192-0001LF, U2 LD39050PU33R

Commit message: Jesus - Updates to header pins on sch
Connections:
- removed net I2C3_SCL1: JP5.4
- removed net I2C3_SDA1: JP5.6
- net I2C1_SCL: now also JP5.1; no longer JP1.6
- net I2C1_SDA: now also JP5.2; no longer JP1.8
- net I2C3_SCL: now also JP5.4
- net I2C3_SDA: now also JP2.2
- net SPI1_MOSI: now also JP1.6; no longer JP1.7
- net SPI1_SCK: now also JP2.4; no longer JP1.2
Changed lines of the file:
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@@
 </segment>
 <segment>
-<pinref part="JP1" gate="A" pin="8"/>
-<wire x1="-111.76" y1="-33.02" x2="-88.9" y2="-33.02" width="0.1524" layer="91"/>
-<label x="-101.6" y="-33.02" size="1.778" layer="95"/>
+<wire x1="-111.76" y1="-71.12" x2="-88.9" y2="-71.12" width="0.1524" layer="91"/>
+<pinref part="JP5" gate="A" pin="2"/>
+<label x="-99.06" y="-71.12" size="1.778" layer="95"/>
 </segment>
 </net>
@@
 </segment>
 <segment>
-<pinref part="JP1" gate="A" pin="6"/>
-<wire x1="-111.76" y1="-30.48" x2="-88.9" y2="-30.48" width="0.1524" layer="91"/>
-<label x="-101.6" y="-30.48" size="1.778" layer="95"/>
+<wire x1="-142.24" y1="-71.12" x2="-119.38" y2="-71.12" width="0.1524" layer="91"/>
+<pinref part="JP5" gate="A" pin="1"/>
+<label x="-139.7" y="-71.12" size="1.778" layer="95"/>
 </segment>
 </net>
@@
 <pinref part="R8" gate="G$1" pin="1"/>
 </segment>
+<segment>
+<wire x1="-111.76" y1="-73.66" x2="-86.36" y2="-73.66" width="0.1524" layer="91"/>
+<pinref part="JP5" gate="A" pin="4"/>
+<label x="-99.06" y="-73.66" size="1.778" layer="95"/>
+</segment>
 </net>
 <net name="I2C3_SDA" class="0">
@@
 <label x="-10.16" y="114.3" size="1.778" layer="95" rot="R90"/>
 <pinref part="R9" gate="G$1" pin="2"/>
+</segment>
+<segment>
+<wire x1="-111.76" y1="-55.88" x2="-88.9" y2="-55.88" width="0.1524" layer="91"/>
+<label x="-101.6" y="-55.88" size="1.778" layer="95"/>
+<pinref part="JP2" gate="A" pin="2"/>
 </segment>
 </net>
@@
 </segment>
 <segment>
-<wire x1="-111.76" y1="-25.4" x2="-88.9" y2="-25.4" width="0.1524" layer="91"/>
-<label x="-101.6" y="-25.4" size="1.778" layer="95"/>
-<pinref part="JP1" gate="A" pin="2"/>
+<wire x1="-111.76" y1="-58.42" x2="-88.9" y2="-58.42" width="0.1524" layer="91"/>
+<label x="-101.6" y="-58.42" size="1.778" layer="95"/>
+<pinref part="JP2" gate="A" pin="4"/>
 </segment>
 </net>
@@
 </segment>
 <segment>
-<wire x1="-119.38" y1="-33.02" x2="-139.7" y2="-33.02" width="0.1524" layer="91"/>
-<label x="-139.7" y="-33.02" size="1.778" layer="95"/>
-<pinref part="JP1" gate="A" pin="7"/>
+<wire x1="-88.9" y1="-30.48" x2="-111.76" y2="-30.48" width="0.1524" layer="91"/>
+<label x="-101.6" y="-30.48" size="1.778" layer="95"/>
+<pinref part="JP1" gate="A" pin="6"/>
 </segment>
 </net>
@@
 </segment>
 </net>
-<net name="I2C3_SCL1" class="0">
-<segment>
-<wire x1="-111.76" y1="-73.66" x2="-86.36" y2="-73.66" width="0.1524" layer="91"/>
-<pinref part="JP5" gate="A" pin="4"/>
-<label x="-99.06" y="-73.66" size="1.778" layer="95"/>
-</segment>
-</net>
-<net name="I2C3_SDA1" class="0">
-<segment>
-<wire x1="-111.76" y1="-76.2" x2="-86.36" y2="-76.2" width="0.1524" layer="91"/>
-<pinref part="JP5" gate="A" pin="6"/>
-<label x="-99.06" y="-76.2" size="1.778" layer="95"/>
-</segment>
-</net>

Commit message: Jesus - Updates to header pins on sch
Parts:
- renumbered BAROMETER to BAR
Connections:
- net EXTI2: now also JP1.2
- net EXTI4: now also JP1.8
- net I2C2_SCL: now also JP1.12; no longer JP1.10
- net I2C2_SDA: now also JP1.10; no longer JP1.12
- net USB_DN: now also JP4.5
- net USB_DP: now also JP4.3
Changed lines of the file:
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@@
 <part name="D1" library="ce-capstone-2022" deviceset="1N5819HW-7-F_1N5819HW-7-F" device=""/>
 <part name="FRAME2" library="frames" library_urn="urn:adsk.eagle:library:229" deviceset="FRAME_C_L" device=""/>
-<part name="BAROMETER" library="DPS310XTSA1" deviceset="DPS310XTSA1" device=""/>
+<part name="BAR" library="DPS310XTSA1" deviceset="DPS310XTSA1" device=""/>
 <part name="GND1" library="supply1" library_urn="urn:adsk.eagle:library:371" deviceset="GND" device=""/>
 <part name="GND8" library="supply1" library_urn="urn:adsk.eagle:library:371" deviceset="GND" device=""/>
@@
 <attribute name="DRAWING_NAME" x="274.32" y="-123.19" size="2.54" layer="94"/>
 </instance>
-<instance part="BAROMETER" gate="G$1" x="-7.62" y="55.88" smashed="yes">
+<instance part="BAR" gate="G$1" x="-7.62" y="55.88" smashed="yes">
 <attribute name="NAME" x="19.05" y="63.5" size="1.778" layer="95" align="center-left"/>
 <attribute name="VALUE" x="-3.81" y="60.96" size="1.778" layer="96" align="center-left"/>
@@
 </segment>
 <segment>
-<pinref part="BAROMETER" gate="G$1" pin="GND_1"/>
+<pinref part="BAR" gate="G$1" pin="GND_1"/>
 <pinref part="GND1" gate="1" pin="GND"/>
 <wire x1="-7.62" y1="48.26" x2="-12.7" y2="48.26" width="0.1524" layer="91"/>
 </segment>
 <segment>
-<pinref part="BAROMETER" gate="G$1" pin="GND_2"/>
+<pinref part="BAR" gate="G$1" pin="GND_2"/>
 <pinref part="GND8" gate="1" pin="GND"/>
 <wire x1="22.86" y1="50.8" x2="35.56" y2="50.8" width="0.1524" layer="91"/>
@@
 </segment>
 <segment>
-<pinref part="BAROMETER" gate="G$1" pin="VDDIO"/>
+<pinref part="BAR" gate="G$1" pin="VDDIO"/>
 <pinref part="L7" gate="A" pin="1"/>
 <wire x1="58.42" y1="38.1" x2="60.96" y2="38.1" width="0.1524" layer="91"/>
@@
 </segment>
 <segment>
-<pinref part="BAROMETER" gate="G$1" pin="SDO"/>
+<pinref part="BAR" gate="G$1" pin="SDO"/>
 <wire x1="22.86" y1="55.88" x2="25.4" y2="55.88" width="0.1524" layer="91"/>
 <label x="22.86" y="55.88" size="1.778" layer="95"/>
 </segment>
 <segment>
-<pinref part="BAROMETER" gate="G$1" pin="CSB"/>
+<pinref part="BAR" gate="G$1" pin="CSB"/>
 <wire x1="-7.62" y1="50.8" x2="-17.78" y2="50.8" width="0.1524" layer="91"/>
 <label x="-15.24" y="50.8" size="1.778" layer="95"/>
@@
 <net name="I2C2_SCL" class="0">
 <segment>
-<pinref part="JP1" gate="A" pin="10"/>
-<wire x1="-111.76" y1="-35.56" x2="-88.9" y2="-35.56" width="0.1524" layer="91"/>
-<label x="-101.6" y="-35.56" size="1.778" layer="95"/>
-</segment>
-<segment>
-<pinref part="BAROMETER" gate="G$1" pin="SCK"/>
+<pinref part="BAR" gate="G$1" pin="SCK"/>
 <wire x1="-7.62" y1="55.88" x2="-15.24" y2="55.88" width="0.1524" layer="91"/>
 <pinref part="R2" gate="G$1" pin="1"/>
@@
 <pinref part="IC1" gate="G$1" pin="PB10"/>
 </segment>
+<segment>
+<wire x1="-88.9" y1="-38.1" x2="-111.76" y2="-38.1" width="0.1524" layer="91"/>
+<label x="-101.6" y="-38.1" size="1.778" layer="95"/>
+<pinref part="JP1" gate="A" pin="12"/>
+</segment>
 </net>
 <net name="I2C2_SDA" class="0">
 <segment>
-<pinref part="JP1" gate="A" pin="12"/>
-<wire x1="-111.76" y1="-38.1" x2="-88.9" y2="-38.1" width="0.1524" layer="91"/>
-<label x="-101.6" y="-38.1" size="1.778" layer="95"/>
-</segment>
-<segment>
-<pinref part="BAROMETER" gate="G$1" pin="SDI"/>
+<pinref part="BAR" gate="G$1" pin="SDI"/>
 <wire x1="-7.62" y1="53.34" x2="-30.48" y2="53.34" width="0.1524" layer="91"/>
 <pinref part="R3" gate="G$1" pin="1"/>
@@
 <label x="203.2" y="-50.8" size="1.778" layer="95" rot="R90"/>
 <pinref part="IC1" gate="G$1" pin="PB11"/>
+</segment>
+<segment>
+<wire x1="-88.9" y1="-35.56" x2="-111.76" y2="-35.56" width="0.1524" layer="91"/>
+<label x="-101.6" y="-35.56" size="1.778" layer="95"/>
+<pinref part="JP1" gate="A" pin="10"/>
 </segment>
 </net>
@@
 <junction x="30.48" y="38.1"/>
 <pinref part="C8" gate="G$1" pin="1"/>
-<pinref part="BAROMETER" gate="G$1" pin="VDD"/>
+<pinref part="BAR" gate="G$1" pin="VDD"/>
 <wire x1="22.86" y1="48.26" x2="30.48" y2="48.26" width="0.1524" layer="91"/>
 <wire x1="30.48" y1="48.26" x2="30.48" y2="38.1" width="0.1524" layer="91"/>
@@
 <wire x1="160.02" y1="167.64" x2="175.26" y2="167.64" width="0.1524" layer="91"/>
 <label x="162.56" y="167.64" size="1.778" layer="95"/>
+</segment>
+<segment>
+<pinref part="JP1" gate="A" pin="2"/>
+<wire x1="-111.76" y1="-25.4" x2="-88.9" y2="-25.4" width="0.1524" layer="91"/>
+<label x="-101.6" y="-25.4" size="1.778" layer="95"/>
 </segment>
 </net>
@@
 <pinref part="IC1" gate="G$1" pin="PA12"/>
 </segment>
+<segment>
+<pinref part="JP4" gate="A" pin="3"/>
+<wire x1="-124.46" y1="33.02" x2="-134.62" y2="33.02" width="0.1524" layer="91"/>
+<label x="-134.62" y="33.02" size="1.778" layer="95"/>
+</segment>
 </net>
 <net name="USB_DN" class="0">
@@
 <label x="220.98" y="10.16" size="1.778" layer="95"/>
 <pinref part="IC1" gate="G$1" pin="PA11"/>
+</segment>
+<segment>
+<pinref part="JP4" gate="A" pin="5"/>
+<wire x1="-124.46" y1="30.48" x2="-134.62" y2="30.48" width="0.1524" layer="91"/>
+<label x="-134.62" y="30.48" size="1.778" layer="95"/>
 </segment>
 </net>
@@
 <label x="162.56" y="147.32" size="1.778" layer="95"/>
 </segment>
-</net>
+<segment>
+<pinref part="JP1" gate="A" pin="8"/>
+<wire x1="-111.76" y1="-33.02" x2="-88.9" y2="-33.02" width="0.1524" layer="91"/>
+<label x="-101.6" y="-33.02" size="1.778" layer="95"/>
+</segment>
+</net>

Commit message: J & N - Added TCXO to sch
Parts:
- added R11: 22, SparkFun-Resistors:22OHM-0402-1/10W-1%
- added Y1: ECS-TXO-3225MV-400-TR, SamacSys_Parts:ECS-TXO-3225MV-400-TR
Connections:
- new net N$3: R11.1, Y1.OUTPUT
- net 3V3: now also Y1.TRI-STATE, Y1.VDD
- net GND: now also Y1.GROUND
- net OSC_IN: now also R11.2
Changed lines of the file:
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@@
 <?xml version="1.0" encoding="utf-8"?>
 <!DOCTYPE eagle SYSTEM "eagle.dtd">
-<eagle version="9.6.2">
+<eagle version="9.4.2">
 <drawing>
 <settings>
@@
 <part name="R17" library="SparkFun-Resistors" library_urn="urn:adsk.eagle:library:532" deviceset="22OHM" device="-0402-1/10W-1%" package3d_urn="urn:adsk.eagle:package:39657/1" value="22"/>
 <part name="R18" library="SparkFun-Resistors" library_urn="urn:adsk.eagle:library:532" deviceset="22OHM" device="-0402-1/10W-1%" package3d_urn="urn:adsk.eagle:package:39657/1" value="22"/>
+<part name="Y1" library="SamacSys_Parts" deviceset="ECS-TXO-3225MV-400-TR" device=""/>
+<part name="GND22" library="supply1" library_urn="urn:adsk.eagle:library:371" deviceset="GND" device=""/>
+<part name="R11" library="SparkFun-Resistors" library_urn="urn:adsk.eagle:library:532" deviceset="22OHM" device="-0402-1/10W-1%" package3d_urn="urn:adsk.eagle:package:39657/1" value="22"/>
 </parts>
 <sheets>
@@
 <attribute name="NAME" x="154.94" y="148.844" size="1.778" layer="95" font="vector" align="bottom-center"/>
 <attribute name="VALUE" x="154.94" y="145.796" size="1.778" layer="96" font="vector" align="top-center"/>
+</instance>
+<instance part="Y1" gate="G$1" x="-12.7" y="-17.78" smashed="yes">
+<attribute name="NAME" x="21.59" y="-10.16" size="1.778" layer="95" align="center-left"/>
+<attribute name="VALUE" x="21.59" y="-12.7" size="1.778" layer="96" align="center-left"/>
+</instance>
+<instance part="GND22" gate="1" x="30.48" y="-27.94" smashed="yes">
+<attribute name="VALUE" x="27.94" y="-30.48" size="1.778" layer="96"/>
+</instance>
+<instance part="R11" gate="G$1" x="50.8" y="-17.78" smashed="yes">
+<attribute name="NAME" x="50.8" y="-16.256" size="1.778" layer="95" font="vector" align="bottom-center"/>
+<attribute name="VALUE" x="50.8" y="-19.304" size="1.778" layer="96" font="vector" align="top-center"/>
 </instance>
 </instances>
@@
 <pinref part="C24" gate="G$1" pin="2"/>
 </segment>
+<segment>
+<pinref part="Y1" gate="G$1" pin="GROUND"/>
+<wire x1="25.4" y1="-20.32" x2="30.48" y2="-20.32" width="0.1524" layer="91"/>
+<wire x1="30.48" y1="-20.32" x2="30.48" y2="-25.4" width="0.1524" layer="91"/>
+<pinref part="GND22" gate="1" pin="GND"/>
+</segment>
 </net>
 <net name="BOOT0" class="0">
@@
 <label x="-35.56" y="210.82" size="1.778" layer="95"/>
 </segment>
+<segment>
+<pinref part="Y1" gate="G$1" pin="VDD"/>
+<wire x1="-12.7" y1="-17.78" x2="-17.78" y2="-17.78" width="0.1524" layer="91"/>
+<wire x1="-17.78" y1="-17.78" x2="-17.78" y2="-15.24" width="0.1524" layer="91"/>
+<label x="-17.78" y="-15.24" size="1.778" layer="95"/>
+</segment>
+<segment>
+<pinref part="Y1" gate="G$1" pin="TRI-STATE"/>
+<wire x1="-12.7" y1="-20.32" x2="-22.86" y2="-20.32" width="0.1524" layer="91"/>
+<wire x1="-22.86" y1="-20.32" x2="-22.86" y2="-27.94" width="0.1524" layer="91"/>
+<label x="-22.86" y="-27.94" size="1.778" layer="95"/>
+</segment>
 </net>
 <net name="USART1_RX" class="0">
@@
 <label x="142.24" y="10.16" size="1.778" layer="95"/>
 </segment>
+<segment>
+<pinref part="R11" gate="G$1" pin="2"/>
+<wire x1="55.88" y1="-17.78" x2="66.04" y2="-17.78" width="0.1524" layer="91"/>
+<label x="60.96" y="-17.78" size="1.778" layer="95"/>
+</segment>
 </net>
 <net name="GPIO_EXTI2" class="0">
@@
 </segment>
 </net>
+<net name="N$3" class="0">
+<segment>
+<pinref part="Y1" gate="G$1" pin="OUTPUT"/>
+<pinref part="R11" gate="G$1" pin="1"/>
+<wire x1="25.4" y1="-17.78" x2="45.72" y2="-17.78" width="0.1524" layer="91"/>
+</segment>
+</net>
