File: PCB/v1/v3/SensorStick.sch (EAGLE design)
At the start: 74 parts, among them U1 TPD4F003DQDR, Y1 ECS-TXO-3225MV-400-TR

Commit message: Jesus - Began to transition GPS to header pins
Parts:
- removed GPS: SAM-M8Q-0-10, SAM-M8Q-0-10:SAM-M8Q-0-10
- removed JP3: (no value), pinhead:PINHD-1X2
- removed JP6: (no value), pinhead:PINHD-1X1
- added JP5: (no value), pinhead:PINHD-2X8
- added R4: 0, SparkFun-Resistors:0OHM-0603-1/10W-5%
Connections:
- removed net N$2: GPS.TIMEPULSE, L4.2
- removed net N$9: C25.2, C28.2, GPS.VCC, L6.1
- new net TIMEPULSE: JP5.6, L4.2
- new net VCC: JP5.1
- new net VCC_GPS: C25.2, C28.2, L6.1
- new net VCC_IO: JP5.7
- new net V_BACKUP: JP5.5
- net 3V3: now also R4.1, R4.2; no longer GPS.VCC_IO, GPS.V_BCKP
- net GND: now also JP5.10, JP5.11, JP5.12, JP5.13, JP5.14, JP5.15, JP5.16, JP5.9; no longer GPS.GND_1, GPS.GND_2, GPS.GND_3, GPS.GND_4, GPS.GND_5, GPS.GND_6, GPS.GND_7, GPS.GND_8, GPS.GND_9
- net GPS_SAFEBOOT: now also JP5.8; no longer GPS.SAFEBOOT_N, JP6.1
- net NRST: now also JP5.3; no longer GPS.RESET_N
- net RX: now also JP5.4; no longer GPS.RXD
- net TX: now also JP5.2; no longer GPS.TXD
- net USART3_RX: no longer JP3.1
- net USART3_TX: no longer JP3.2

Commit message: Jesus - Cleaning up GPS schematic
Other:
- moved on the sheet: C25, C28, C29, JP5, L2, L4, L5, L6, R4

Commit message: Jesus - Further updates to Mag/GPS/USART breakout
Parts:
- removed C10, C11: 0.1uF, SparkFun-Capacitors:0.1UF-0402-6.3V-10%-X7R
- removed C12: 10uF, SparkFun-Capacitors:10UF-0603-6.3V-20%
- removed C13: 0.22uF, SparkFun-Capacitors:0.22UF-0603-25V-10%
- removed C25, C27: 4.7uF, SparkFun-Capacitors:4.7UF0603
- removed C28, C29: 0.1uF, SparkFun-Capacitors:0.1UF-0402-16V-10%
- removed JP1: (no value), pinhead:PINHD-1X7
- removed JP2: (no value), pinhead:PINHD-1X6
- removed JP4: (no value), pinhead:PINHD-1X3
- removed JP5: (no value), pinhead:PINHD-2X8
- removed L2, L4, L5, L6, L8: BLM03AG601SN1D, BLM03AG601SN1D:BLM03AG601SN1D
- removed MAGNETOMETER: IIS2MDCTR, IIS2MDCTR:IIS2MDCTR
- removed R4: 0, SparkFun-Resistors:0OHM-0603-1/10W-5%
- added SV1, SV2: (no value), con-lsta:FE05-1
Connections:
- removed net GPS_SAFEBOOT: JP5.8
- removed net N$10: C11.1, C12.1, C27.1, L8.1, MAGNETOMETER.VDD
- removed net N$7: C13.1, MAGNETOMETER.C1
- removed net RX: JP5.4, L5.2
- removed net SPI2_MISO: JP4.2, MICROCONTROLLER.PB14
- removed net SPI2_MOSI: JP4.1, MICROCONTROLLER.PB15
- removed net SPI2_SCK: JP4.3, MICROCONTROLLER.PB13
- removed net TIMEPULSE: JP5.6, L4.2
- removed net TX: JP5.2, L2.2
- removed net VCC: JP5.1
- removed net VCC_GPS: C25.2, C28.2, L6.1
- removed net VCC_IO: JP5.7
- removed net V_BACKUP: JP5.5
- new net USART2_RX: MICROCONTROLLER.PA3, SV1.3
- new net USART2_TX: MICROCONTROLLER.PA2, SV1.2
- net 3V3: now also SV1.5, SV2.5; no longer AIRSPEED.VCC, C10.1, C29.2, C3.2, JP2.1, L6.2, L8.2, MAGNETOMETER.CS, MAGNETOMETER.VDD_IO, R4.1, R4.2
- net 5V: now also AIRSPEED.VCC, C3.2; no longer JP1.1
- net EXTI4: now also SV2.1; no longer MAGNETOMETER.INT/DRDY
- net GND: now also SV1.4, SV2.4; no longer C10.2, C11.2, C12.2, C13.2, C25.1, C27.2, C28.1, C29.1, JP1.2, JP2.2, JP5.10, JP5.11, JP5.12, JP5.13, JP5.14, JP5.15, JP5.16, JP5.9, MAGNETOMETER.GND_1, MAGNETOMETER.GND_2
- net GPIO_EXTI1: now also SV1.1; no longer L4.1
- net I2C1_SCL: now also SV2.3; no longer JP2.6, MAGNETOMETER.SCL/SPC
- net I2C1_SDA: now also SV2.2; no longer JP2.5, MAGNETOMETER.SDA/SDI/SDO
- net I2C2_SCL: no longer JP1.4
- net I2C2_SDA: no longer JP1.3
- net I2C3_SCL: no longer JP2.4
- net I2C3_SDA: no longer JP2.3
- net NRST: no longer JP5.3
- net SPI1_MISO: no longer JP1.6
- net SPI1_MOSI: no longer JP1.5
- net SPI1_SCK: no longer JP1.7
- net USART3_RX: no longer L5.1
- net USART3_TX: no longer L2.1
Other:
- moved on the sheet: AIRSPEED, C3, R6, R7, R8, R9

Commit message: Jesus - Cleaned up sch/layout, finished
Parts:
- removed SV2: (no value), con-lsta:FE05-1
- added IC1: (no value), ic-package:DIL24-3
- added JP1: (no value), pinhead:PINHD-2X3
Connections:
- net 3V3: now also JP1.1, JP1.3; no longer SV2.5
- net EXTI4: now also JP1.6; no longer SV2.1
- net GND: now also JP1.5; no longer SV2.4
- net I2C1_SCL: now also JP1.2; no longer SV2.3
- net I2C1_SDA: now also JP1.4; no longer SV2.2
Other:
- moved on the sheet: AIRSPEED, BAROMETER, C1, C14, C15, C16, C17, C18, C19, C2, C20, C21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

Commit message: Jesus - Removed DIL24 IC connector
Parts:
- removed IC1: (no value), ic-package:DIL24-3
Changed lines of the file:
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@@
 <part name="U1" library="TPD4F003DQDR" deviceset="TPD4F003DQDR" device=""/>
 <part name="SV1" library="con-lsta" library_urn="urn:adsk.eagle:library:161" deviceset="FE05-1" device="" package3d_urn="urn:adsk.eagle:package:8190/1"/>
-<part name="IC1" library="ic-package" library_urn="urn:adsk.eagle:library:239" deviceset="DIL24" device="-3" package3d_urn="urn:adsk.eagle:package:3299/3"/>
 <part name="JP1" library="pinhead" library_urn="urn:adsk.eagle:library:325" deviceset="PINHD-2X3" device="" package3d_urn="urn:adsk.eagle:package:22462/2"/>
 <part name="FRAME1" library="frames" library_urn="urn:adsk.eagle:library:229" deviceset="DINA3_L" device=""/>
@@
 <attribute name="NAME" x="123.19" y="125.222" size="1.778" layer="95"/>
 </instance>
-<instance part="IC1" gate="G$1" x="203.2" y="139.7" smashed="yes" rot="R90">
-<attribute name="NAME" x="186.055" y="135.255" size="1.778" layer="95" rot="R90"/>
-<attribute name="VALUE" x="219.71" y="135.255" size="1.778" layer="96" rot="R90"/>
-</instance>
 <instance part="JP1" gate="A" x="200.66" y="116.84" smashed="yes">
