File: PCB/v1/v3/SensorStick_v3_noah.brd (EAGLE design)
At the start: 76.2 x 38.1 mm, 56 parts, among them U1 TPD4F003DQDR, Y1 ECS-TXO-3225MV-400-TR

Commit message: Add files via upload
Parts:
- moved SV1 0.25 mm to (66.0, 30.0), turned to 270 degrees
Routing:
- net GPIO_EXTI1: track 54.0 -> 50.4 mm
- net GND: track 114.3 -> 117.3 mm, vias 27 -> 28
- net USART2_TX: track 49.9 -> 47.5 mm, vias 2 -> 4
- net 3V3: track 98.8 -> 100.3 mm
- net USART2_RX: track 52.4 -> 53.2 mm
Other:
- board size 76.2 x 38.1 mm -> 71.4 x 38.4 mm
Changed lines of the file:
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@@
 <board>
 <plain>
-<wire x1="0" y1="0" x2="76.2" y2="0" width="0" layer="20"/>
-<wire x1="76.2" y1="0" x2="76.2" y2="38.1" width="0" layer="20"/>
-<wire x1="76.2" y1="38.1" x2="0" y2="38.1" width="0" layer="20"/>
-<wire x1="0" y1="38.1" x2="0" y2="0" width="0" layer="20"/>
-<text x="44.704" y="33.782" size="0.762" layer="21">IMU</text>
-<text x="52.07" y="25.908" size="1.27" layer="21" rot="R180">AIR</text>
+<wire x1="0" y1="0" x2="71.374" y2="0" width="0" layer="20"/>
+<wire x1="71.374" y1="0" x2="71.374" y2="38.354" width="0" layer="20"/>
+<wire x1="71.374" y1="38.354" x2="0" y2="38.354" width="0" layer="20"/>
+<wire x1="0" y1="38.354" x2="0" y2="0" width="0" layer="20"/>
+<text x="38.862" y="26.67" size="0.762" layer="21">IMU</text>
+<text x="54.356" y="29.21" size="1.27" layer="21" rot="R180">AIR</text>
 <text x="18.288" y="33.782" size="0.762" layer="21">BAR</text>
-<text x="63.754" y="36.576" size="0.762" layer="21" rot="R180">GPS</text>
+<text x="64.008" y="36.322" size="0.762" layer="21" rot="R180">GPS</text>
 <text x="17.78" y="6.604" size="0.508" layer="21" rot="R270">BOOT0</text>
 <text x="29.21" y="1.778" size="0.508" layer="21" rot="R270">RST</text>
@@
 Marko Ristic
 Danny Cardenas</text>
-<text x="72.644" y="16.256" size="1.016" layer="21">1</text>
 <text x="50.8" y="22.606" size="1.016" layer="21" rot="R270">1</text>
 <text x="9.398" y="0.762" size="0.254" layer="21">⠀⠀⠀⠀⠀⠀⢀⣀⣀⠀⠀⠀⠀⠀⠀⠀⠀⠀⠀⠀⠀⠀⠀⠀⠀⠀⠀⠀⠀⠀
@@
 </element>
 <element name="R9" library="SparkFun-Resistors" library_urn="urn:adsk.eagle:library:532" package="0603" package3d_urn="urn:adsk.eagle:package:39650/1" value="4.7k" x="62.992" y="1.016" smashed="yes" rot="R180">
-<attribute name="NAME" x="63.754" y="0" size="0.3048" layer="25" font="vector" ratio="20" rot="R180" align="bottom-center"/>
+<attribute name="NAME" x="63.246" y="2.032" size="0.3048" layer="25" font="vector" ratio="20" rot="R180" align="bottom-center"/>
 <attribute name="PROD_ID" value="RES-07857" x="62.992" y="1.016" size="1.778" layer="27" rot="R180" display="off"/>
 </element>
@@
 <attribute name="MFR_NAME" value="Texas Instruments" x="18.034" y="9.906" size="1.778" layer="27" rot="R180" display="off"/>
 </element>
-<element name="SV1" library="con-lsta" library_urn="urn:adsk.eagle:library:161" package="FE05-1" package3d_urn="urn:adsk.eagle:package:8190/1" value="" x="66.294" y="29.972" smashed="yes" rot="R90">
-<attribute name="MF" value="" x="66.294" y="29.972" size="1.778" layer="27" rot="R90" display="off"/>
-<attribute name="MPN" value="" x="66.294" y="29.972" size="1.778" layer="27" rot="R90" display="off"/>
-<attribute name="OC_FARNELL" value="unknown" x="66.294" y="29.972" size="1.778" layer="27" rot="R90" display="off"/>
-<attribute name="OC_NEWARK" value="unknown" x="66.294" y="29.972" size="1.778" layer="27" rot="R90" display="off"/>
-<attribute name="VALUE" x="64.643" y="29.972" size="1.27" layer="27" ratio="10" rot="R90"/>
+<element name="SV1" library="con-lsta" library_urn="urn:adsk.eagle:library:161" package="FE05-1" package3d_urn="urn:adsk.eagle:package:8190/1" value="" x="66.04" y="29.972" smashed="yes" rot="R270">
+<attribute name="MF" value="" x="66.04" y="29.972" size="1.778" layer="27" rot="R270" display="off"/>
+<attribute name="MPN" value="" x="66.04" y="29.972" size="1.778" layer="27" rot="R270" display="off"/>
+<attribute name="OC_FARNELL" value="unknown" x="66.04" y="29.972" size="1.778" layer="27" rot="R270" display="off"/>
+<attribute name="OC_NEWARK" value="unknown" x="66.04" y="29.972" size="1.778" layer="27" rot="R270" display="off"/>
+<attribute name="VALUE" x="67.691" y="29.972" size="1.27" layer="27" ratio="10" rot="R270"/>
 </element>
 <element name="IC2" library="ic-package" library_urn="urn:adsk.eagle:library:239" package="DIL24-6" package3d_urn="urn:adsk.eagle:package:1009/2" value="" x="55.626" y="11.176" smashed="yes" rot="R180">
@@
 <via x="4.318" y="27.178" extent="1-16" drill="0.35"/>
 <polygon width="0.1524" layer="15">
-<vertex x="0" y="38.1"/>
-<vertex x="76.2" y="38.1"/>
-<vertex x="76.2" y="0"/>
+<vertex x="0" y="38.354"/>
+<vertex x="71.374" y="38.354"/>
+<vertex x="71.374" y="0"/>
 <vertex x="0" y="0"/>
 </polygon>
@@
 <wire x1="48.768" y1="25.742" x2="48.768" y2="26.162" width="0.3048" layer="1"/>
 <via x="48.768" y="26.162" extent="1-16" drill="0.35"/>
-<via x="68.58" y="35.052" extent="1-16" drill="0.35"/>
-<wire x1="66.294" y1="35.052" x2="68.58" y2="35.052" width="0.2032" layer="1"/>
+<wire x1="66.04" y1="24.892" x2="69.85" y2="24.892" width="0.2032" layer="1"/>
+<via x="69.85" y="24.892" extent="1-16" drill="0.35"/>
 </signal>
 <signal name="USART1_RX">
@@
 <contactref element="IMU" pad="7"/>
 <polygon width="0.1524" layer="2">
-<vertex x="0" y="38.1"/>
-<vertex x="76.2" y="38.1"/>
-<vertex x="76.2" y="0"/>
+<vertex x="0" y="38.354"/>
+<vertex x="71.374" y="38.354"/>
+<vertex x="71.374" y="0"/>
 <vertex x="0" y="0"/>
 </polygon>
@@
 <wire x1="49.475" y1="32.965" x2="49.53" y2="33.02" width="0.3048" layer="1"/>
 <via x="49.53" y="33.02" extent="1-16" drill="0.35"/>
+<wire x1="66.04" y1="27.432" x2="69.088" y2="27.432" width="0.2032" layer="1"/>
+<via x="69.088" y="27.432" extent="1-16" drill="0.35"/>
 </signal>
 <signal name="I2C2_SCL">
@@
 <wire x1="40.9224" y1="35.5884" x2="44.1676" y2="35.5884" width="0.2032" layer="16"/>
 <wire x1="44.1676" y1="35.5884" x2="45.72" y2="34.036" width="0.2032" layer="16"/>
-<wire x1="45.72" y1="34.036" x2="47.244" y2="34.036" width="0.2032" layer="16"/>
-<via x="47.244" y="34.036" extent="1-16" drill="0.35"/>
-<wire x1="62.02329375" y1="28.3764" x2="62.8096" y2="28.3764" width="0.2032" layer="1"/>
-<wire x1="62.8096" y1="28.3764" x2="66.294" y2="24.892" width="0.2032" layer="1"/>
-<wire x1="47.244" y1="34.036" x2="56.36369375" y2="34.036" width="0.2032" layer="1"/>
-<wire x1="56.36369375" y1="34.036" x2="62.02329375" y2="28.3764" width="0.2032" layer="1"/>
+<wire x1="45.72" y1="34.036" x2="60.452" y2="34.036" width="0.2032" layer="16"/>
+<wire x1="60.452" y1="34.036" x2="61.468" y2="35.052" width="0.2032" layer="16"/>
+<wire x1="61.468" y1="35.052" x2="62.738" y2="35.052" width="0.2032" layer="16"/>
+<via x="62.738" y="35.052" extent="1-16" drill="0.35"/>
+<wire x1="62.738" y1="35.052" x2="66.04" y2="35.052" width="0.2032" layer="1"/>
 </signal>
 <signal name="GPIO_EXTI3">
@@
 <wire x1="45.212" y1="36.068" x2="46.228" y2="35.052" width="0.2032" layer="16"/>
 <via x="46.228" y="35.052" extent="1-16" drill="0.35"/>
-<wire x1="46.228" y1="35.052" x2="58.674" y2="35.052" width="0.2032" layer="1"/>
-<wire x1="58.674" y1="35.052" x2="66.294" y2="27.432" width="0.2032" layer="1"/>
+<wire x1="46.228" y1="35.052" x2="59.944" y2="35.052" width="0.2032" layer="1"/>
+<wire x1="59.944" y1="35.052" x2="61.468" y2="33.528" width="0.2032" layer="1"/>
+<via x="61.468" y="33.528" extent="1-16" drill="0.35"/>
+<wire x1="61.468" y1="33.528" x2="63.246" y2="33.528" width="0.2032" layer="16"/>
+<wire x1="63.246" y1="33.528" x2="64.008" y2="32.766" width="0.2032" layer="16"/>
+<via x="64.008" y="32.766" extent="1-16" drill="0.35"/>
+<wire x1="64.008" y1="32.766" x2="65.786" y2="32.766" width="0.2032" layer="1"/>
+<wire x1="65.786" y1="32.766" x2="66.04" y2="32.512" width="0.2032" layer="1"/>
 </signal>
 <signal name="USART2_RX">
@@
 <via x="45.974" y="36.322" extent="1-16" drill="0.35"/>
 <wire x1="45.974" y1="36.322" x2="59.944" y2="36.322" width="0.2032" layer="1"/>
-<wire x1="59.944" y1="36.322" x2="66.294" y2="29.972" width="0.2032" layer="1"/>
 <wire x1="28.702" y1="27.178" x2="29.718" y2="27.178" width="0.2032" layer="1"/>
 <wire x1="29.718" y1="27.178" x2="29.972" y2="27.432" width="0.2032" layer="1"/>
@@
 <wire x1="29.718" y1="36.576" x2="45.72" y2="36.576" width="0.2032" layer="16"/>
 <wire x1="45.72" y1="36.576" x2="45.974" y2="36.322" width="0.2032" layer="16"/>
+<wire x1="59.944" y1="36.322" x2="62.484" y2="33.782" width="0.2032" layer="1"/>
+<wire x1="62.484" y1="33.782" x2="62.484" y2="32.004" width="0.2032" layer="1"/>
+<wire x1="62.484" y1="32.004" x2="64.516" y2="29.972" width="0.2032" layer="1"/>
+<wire x1="64.516" y1="29.972" x2="66.04" y2="29.972" width="0.2032" layer="1"/>
 </signal>
 </signals>
